File: girlvoice.kicad_sch (KiCad schematic)
At the start: 148 parts, among them J1 IPS 1.28 inch SPI GC9A01, J2 Pico, J3 PAJ7620F2, J7 USB_C, J8 AudioJack 2.5mm, Q1 BSS214NW, Q2 AO3401A, SW1 ON/OFF, SW2 UP, SW3 DOWN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

Commit message: ADD: Manufacturing files
Other:
- note added: "I2C: 0x15"
